Commit message: 2025.11.13: 优化被抓物体会被打飞的现象

File: source/isaaclab_tasks/isaaclab_tasks/manager_based/manipulation/lift/robot_model/arm_description/urdf/R50/r50_v6_rev.urdf (robot description, URDF)
Before this commit: robot 00_r50_arm_2_7_asm_09059.SLDASM, 15 links, 14 joints
Links:
- removed link M6_1_1_LINK
- removed link M6_2_2_LINK
Joints:
- removed joint M6_1_1
- removed joint M6_2_2
