Commit message: 2025.12.17: 抓取红色车(没有随机化材质))

File: source/isaaclab_tasks/isaaclab_tasks/manager_based/manipulation/lift/robot_model/arm_description/urdf/R50/r50_v5.urdf (robot description, URDF)
Before this commit: robot 00_r50_arm_2_7_asm_09059.SLDASM, 15 links, 14 joints
Joints:
- joint M0: limit (none) -> lower=-1.57 upper=1.57 effort=0 velocity=0; type fixed -> continuous
- joint M3: limit lower=3. upper=5.2 effort=100 velocity=5 -> lower=3. upper=5。2 effort=100 velocity=5
- joint M5: limit lower=0 upper=0 effort=100 velocity=5 -> lower=-2.4422 upper=3.1416 effort=100 velocity=5

Commit message: 2025.12.24: 稳定抓取多个物体(lego/bus/paper)

File: source/isaaclab_tasks/isaaclab_tasks/manager_based/manipulation/lift/robot_model/arm_description/urdf/R50/r50_v5.urdf (robot description, URDF)
Before this commit: robot 00_r50_arm_2_7_asm_09059.SLDASM, 15 links, 14 joints
Joints:
- joint M0: limit lower=-1.57 upper=1.57 effort=0 velocity=0 -> (none); type continuous -> fixed
- joint M3: limit lower=3. upper=5。2 effort=100 velocity=5 -> lower=3. upper=5.2 effort=100 velocity=5
- joint M5: limit lower=-2.4422 upper=3.1416 effort=100 velocity=5 -> lower=0 upper=0 effort=100 velocity=5
